File: Caon-Handwired-Prototype.kicad_pcb (KiCad board)
At the start: 2 copper layers, 4 parts, among them U1 74HC595, U2 SuperMini nRF52840

Commit message: Update
Parts:
- added ENC_R1: 10k, Resistor_THT:R_Axial_DIN0204_L3.6mm_D1.6mm_P2.54mm_Vertical, F.Cu at (127.0, 76.2)
- added ENC_R2: 10k, Resistor_THT:R_Axial_DIN0204_L3.6mm_D1.6mm_P2.54mm_Vertical, F.Cu at (127.0, 79.3)
- added ENC_R3: 10k, Resistor_THT:R_Axial_DIN0204_L3.6mm_D1.6mm_P2.54mm_Vertical, F.Cu at (127.0, 82.5)
- added ENC_R4: 10k, Resistor_THT:R_Axial_DIN0204_L3.6mm_D1.6mm_P2.54mm_Vertical, F.Cu at (127.0, 85.7)
- added SW1: EC11 ENCODER 1, PCM_marbastlib-various:ROT_Alps_EC11E-Switch, F.Cu at (137.2, 50.9)
- added SW2: EC11 ENCODER 2, PCM_marbastlib-various:ROT_Alps_EC11E-Switch, F.Cu at (152.4, 50.9)
- added S_D3: ~, Caon_Footprint:D_DO-35_SOD27_P2.54mm_Caon65, F.Cu at (99.1, 54.6)
- added S_D4: ~, Caon_Footprint:D_DO-35_SOD27_P2.54mm_Caon65, F.Cu at (99.1, 58.4)
- added U3: 74HC595, Package_DIP:DIP-16_W7.62mm, F.Cu at (66.0, 94.0)
- S_D1, S_D2: value 1N4148 -> ~; footprint Diode_THT:D_DO-35_SOD27_P2.54mm_Vertical_AnodeUp -> Caon_Footprint:D_DO-35_SOD27_P2.54mm_Caon65
- moved S_D2 26.1 mm to (99.1, 50.9)
- moved S_D1 25.0 mm to (99.1, 47.1)
- moved U1 17.8 mm to (66.0, 71.1)
- moved U2 17.8 mm to (68.6, 52.1)
Connections:
- S_D1 pad 1: (no net) -> C1
- S_D1 pad 2: (no net) -> Net-(S_D1-A)
- S_D2 pad 1: (no net) -> C2
- S_D2 pad 2: (no net) -> Net-(S_D2-A)

Commit message: Schematic update
Parts:
- added D1: ~, Caon_Footprint:D_DO-35_SOD27_P2.54mm_Caon65, F.Cu at (170.2, 72.7)
- added D2: ~, Caon_Footprint:D_DO-35_SOD27_P2.54mm_Caon65, F.Cu at (170.2, 76.4)
- added D3: ~, Caon_Footprint:D_DO-35_SOD27_P2.54mm_Caon65, F.Cu at (170.2, 80.2)
- added D4: ~, Caon_Footprint:D_DO-35_SOD27_P2.54mm_Caon65, F.Cu at (170.2, 84.0)
- added D5: ~, Caon_Footprint:D_DO-35_SOD27_P2.54mm_Caon65, F.Cu at (170.2, 87.7)
- added D6: ~, Caon_Footprint:D_DO-35_SOD27_P2.54mm_Caon65, F.Cu at (170.2, 91.5)
- added D7: ~, Caon_Footprint:D_DO-35_SOD27_P2.54mm_Caon65, F.Cu at (170.2, 95.3)
- added D8: ~, Caon_Footprint:D_DO-35_SOD27_P2.54mm_Caon65, F.Cu at (170.2, 99.1)
- added SW3: SW_PUSH_MX, Caon_Footprint:SW_PUSH_6mm, F.Cu at (164.2, 74.6)
- added SW4: EC11 ENCODER 1, PCM_marbastlib-various:ROT_Alps_EC11E-Switch, F.Cu at (111.8, 109.3)
- added SW5: SW_PUSH_MX, Caon_Footprint:SW_PUSH_6mm, F.Cu at (164.2, 82.2)
- added SW6: SW_PUSH_MX, Caon_Footprint:SW_PUSH_6mm, F.Cu at (164.2, 89.8)
- added SW7: SW_PUSH_MX, Caon_Footprint:SW_PUSH_6mm, F.Cu at (164.2, 97.4)
- added SW8: EC11 ENCODER 1, PCM_marbastlib-various:ROT_Alps_EC11E-Switch, F.Cu at (127.0, 109.3)
- SW1: value EC11 ENCODER 1 -> SW_PUSH_MX; footprint PCM_marbastlib-various:ROT_Alps_EC11E-Switch -> Caon_Footprint:SW_PUSH_6mm
- SW2: value EC11 ENCODER 2 -> SW_PUSH_MX; footprint PCM_marbastlib-various:ROT_Alps_EC11E-Switch -> Caon_Footprint:SW_PUSH_6mm
- U2: value SuperMini nRF52840 -> 74HC595; footprint Caon_Footprint:SuperMini_NiceNano_USBdn -> Package_DIP:DIP-16_W7.62mm
- U3: value 74HC595 -> SuperMini nRF52840; footprint Package_DIP:DIP-16_W7.62mm -> Caon_Footprint:SuperMini_NiceNano_USBdn
Connections:
- S_D2 pad 1: C2 -> C3
- S_D3 pad 1: C3 -> C2
- U1 pad 13: GND -> ENC1_A
- U1 pad 7: Net-(S_D2-A) -> Net-(S_D3-A)
- U1 pad 8: GND -> ENC1_A
- U2 pad 1: MOSI -> unconnected-(U2-QB-Pad1)
- U2 pad 10: unconnected-(U2-P0.11-Pad10) -> +3V3
- U2 pad 11: ENC1_A -> SCK
- U2 pad 12: ENC1_B -> CS
- U2 pad 13: unconnected-(U2-BAT+-Pad13) -> ENC1_A
- U2 pad 14: GND -> MOSI
- U2 pad 2: SCK -> unconnected-(U2-QC-Pad2)
- U2 pad 3: GND -> unconnected-(U2-QD-Pad3)
- U2 pad 4: GND -> unconnected-(U2-QE-Pad4)
- U2 pad 5: CS -> unconnected-(U2-QF-Pad5)
- U2 pad 6: unconnected-(U2-P0.20-Pad6) -> Net-(S_D2-A)
- U2 pad 7: unconnected-(U2-P0.22-Pad7) -> Net-(S_D4-A)
- U2 pad 8: unconnected-(U2-P0.24-Pad8) -> ENC1_A
- U3 pad 1: unconnected-(U3-QB-Pad1) -> MOSI
- U3 pad 10: +3V3 -> unconnected-(U3-P0.11-Pad10)
- U3 pad 11: SCK -> ENC1_A
- U3 pad 12: CS -> ENC1_B
- U3 pad 13: GND -> unconnected-(U3-BAT+-Pad13)
- U3 pad 14: MOSI -> ENC1_A
- U3 pad 2: unconnected-(U3-QC-Pad2) -> SCK
- U3 pad 3: unconnected-(U3-QD-Pad3) -> ENC1_A
- U3 pad 4: unconnected-(U3-QE-Pad4) -> ENC1_A
- U3 pad 5: unconnected-(U3-QF-Pad5) -> CS
- U3 pad 6: Net-(S_D3-A) -> unconnected-(U3-P0.20-Pad6)
- U3 pad 7: Net-(S_D4-A) -> unconnected-(U3-P0.22-Pad7)
- U3 pad 8: GND -> unconnected-(U3-P0.24-Pad8)

Commit message: Update
Parts:
- SW1, SW2, SW3, SW5, SW6, SW7: value SW_PUSH_MX -> ~
- moved SW6 81.2 mm to (83.8, 78.7), turned to 90 degrees
- moved U2 65.9 mm to (40.6, 111.8)
- moved U3 33.2 mm to (43.2, 69.8)
- moved U1 31.0 mm to (40.6, 88.9)
Connections:
- SW1 pad 1: Net-(D1-A) -> C0
- SW1 pad 2: C0 -> Net-(D1-A)
- SW2 pad 1: Net-(D2-A) -> C1
- SW2 pad 2: C1 -> Net-(D2-A)
- SW3 pad 1: Net-(D3-A) -> C2
- SW3 pad 2: C2 -> Net-(D3-A)
- SW4 pad MP: ENC1_A -> unconnected-(SW4-PadMP)_1
- SW5 pad 1: Net-(D5-A) -> C0
- SW5 pad 2: C0 -> Net-(D5-A)
- SW6 pad 1: Net-(D6-A) -> C1
- SW6 pad 2: C1 -> Net-(D6-A)
- SW7 pad 1: Net-(D7-A) -> C2
- SW7 pad 2: C2 -> Net-(D7-A)
- SW8 pad MP: ENC1_A -> unconnected-(SW8-PadMP)
Routing:
- net ENC1_A: track 0.00 -> 168.9 mm, vias 0 -> 9
- net +3V3: track 0.00 -> 129.7 mm, vias 0 -> 16
- net SCK: track 0.00 -> 99.7 mm, vias 0 -> 3
- net CS: track 0.00 -> 91.4 mm, vias 0 -> 3
- net MOSI: track 0.00 -> 86.4 mm, vias 0 -> 4

Commit message: update
Parts:
- moved SW3 156.7 mm to (27.9, 151.9), turned to -90 degrees
- moved SW2 155.6 mm to (27.9, 144.3), turned to -90 degrees
- moved SW1 138.9 mm to (27.9, 136.6), turned to -90 degrees
- moved SW5 129.3 mm to (50.8, 144.3), turned to 90 degrees
- moved SW7 125.8 mm to (50.8, 151.9), turned to -90 degrees
- moved SW8 116.8 mm to (38.0, 184.9), turned to -90 degrees
- moved SW4 93.7 mm to (38.0, 167.1), turned to -90 degrees
- moved SW6 66.6 mm to (50.8, 136.6), turned to -90 degrees
- moved U1 5.11 mm to (35.6, 88.4)
- moved U2 5.11 mm to (35.6, 111.2)
- moved U3 5.11 mm to (38.1, 69.3)

Commit message: Update
Parts:
- moved D3 159.4 mm to (30.5, 157.0), turned to -90 degrees
- moved D2 156.4 mm to (30.5, 146.8), turned to -90 degrees
- moved D1 153.7 mm to (30.5, 136.6), turned to -90 degrees
- moved D8 151.8 mm to (48.3, 189.5), turned to -90 degrees
- moved D4 150.2 mm to (48.3, 171.7), turned to -90 degrees
- moved D7 136.6 mm to (48.3, 157.0), turned to -90 degrees
- moved D6 133.9 mm to (48.3, 146.8), turned to -90 degrees
- moved D5 131.4 mm to (48.3, 136.6), turned to -90 degrees
- moved S_D2 98.4 mm to (27.9, 118.9)
- moved S_D4 95.0 mm to (27.9, 121.4)
- moved S_D1 89.8 mm to (25.4, 98.5)
- moved S_D3 87.1 mm to (25.4, 101.1)
- moved ENC_R1 61.2 mm to (78.7, 113.8), turned to 90 degrees
- moved ENC_R2 50.9 mm to (81.3, 101.7)
- moved ENC_R3 50.9 mm to (81.3, 104.8)
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Connections:
- S_D3 pad 1: C2 -> C0
- S_D4 pad 1: C4 -> C2
Routing:
- net Net-(D3-A): track 0.00 -> 5.08 mm
- net Net-(D2-A): track 0.00 -> 5.08 mm
- net Net-(D1-A): track 0.00 -> 5.08 mm
- net Net-(D7-A): track 0.00 -> 5.08 mm
- net Net-(D6-A): track 0.00 -> 5.08 mm
- net Net-(D5-A): track 0.00 -> 5.08 mm
- net R1: track 0.00 -> 3.31 mm
- net Net-(D4-A): track 0.00 -> 3.31 mm

Commit message: Schematic Update
Parts:
- added REF**: Standard 830 Breadboard, Caon_Footprint:Standard 830 Breadboard, F.Cu at (-33.0, 32.5)
- moved SW1 77.4 mm to (106.7, 106.2), turned to 90 degrees
- moved SW2 77.4 mm to (106.7, 116.3), turned to 90 degrees
- moved SW3 77.4 mm to (106.7, 126.5), turned to 90 degrees
- moved D1 77.4 mm to (101.6, 106.2), turned to 90 degrees
- moved D2 77.4 mm to (101.6, 116.3), turned to 90 degrees
- moved D3 77.4 mm to (101.6, 126.5), turned to 90 degrees
- moved S_D1 61.9 mm to (83.8, 118.9), turned to -90 degrees
- moved U1 61.4 mm to (88.9, 57.9)
- moved U2 61.4 mm to (88.9, 80.8)
- moved SW4 61.1 mm to (91.2, 141.7), turned to 90 degrees
- moved SW8 61.1 mm to (91.2, 159.5), turned to 90 degrees
- moved U3 60.2 mm to (91.4, 41.4)
- moved S_D2 59.1 mm to (81.3, 144.3), turned to 90 degrees
- moved S_D3 58.9 mm to (83.8, 108.7), turned to -90 degrees
- moved ENC_R4 57.7 mm to (101.6, 162.0), turned to -90 degrees
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Connections:
- SW4 pad C: ENC1_A -> GND
- SW8 pad C: ENC1_A -> GND
- U1 pad 13: ENC1_A -> GND
- U1 pad 8: ENC1_A -> GND
- U2 pad 13: ENC1_A -> GND
- U2 pad 8: ENC1_A -> GND
- U3 pad 14: ENC1_A -> GND
- U3 pad 28: ENC1_A -> GND
- U3 pad 3: ENC1_A -> GND
- U3 pad 4: ENC1_A -> GND
Routing:
- net GND: track 0.00 -> 402.1 mm, vias 0 -> 4
- net +3V3: track 129.7 -> 342.9 mm, vias 16 -> 8
- net ENC1_B: track 0.00 -> 102.7 mm, vias 0 -> 2
- net R1: track 3.31 -> 66.0 mm, vias 0 -> 3
- net ENC1_A: track 168.9 -> 112.3 mm, vias 9 -> 2
- net R0: track 0.00 -> 55.9 mm, vias 0 -> 3
- net C2: track 0.00 -> 27.9 mm, vias 0 -> 2
- net C1: track 0.00 -> 27.9 mm, vias 0 -> 2
- net C0: track 0.00 -> 27.9 mm, vias 0 -> 2
- net CS: track 91.4 -> 83.2 mm, vias 3 -> 0
- net SCK: track 99.7 -> 91.4 mm, vias 3 -> 0
- net MOSI: track 86.4 -> 78.7 mm, vias 4 -> 0
- net ENC2_B: track 0.00 -> 5.48 mm, vias 0 -> 1
- net ENC2_A: track 0.00 -> 5.48 mm, vias 0 -> 1
- net Net-(D8-A): track 0.00 -> 2.97 mm
Other:
- copper layers 2 -> 6

Commit message: Schematic update
Parts:
- removed REF**: Standard 830 Breadboard, Caon_Footprint:Standard 830 Breadboard
Connections:
- U3 pad 17: Row 0 -> R0
- U3 pad 18: Row 1 -> R1
Routing:
- net ENC2_A: track 5.48 -> 175.7 mm
- net ENC2_B: track 5.48 -> 152.8 mm
- net R0: track 55.9 -> 191.5 mm
- net R1: track 66.0 -> 198.1 mm
- net Net-(S_D1-A): track 0.00 -> 79.2 mm
- net Net-(S_D2-A): track 0.00 -> 69.9 mm
- net Net-(S_D3-A): track 0.00 -> 65.0 mm
- net Net-(S_D4-A): track 0.00 -> 58.4 mm
- net C3: track 0.00 -> 28.7 mm
- net GND: track 402.1 -> 404.6 mm

Commit message: bump version to V0.1
Parts:
- added REF**: Standard 830 Breadboard, Caon_Footprint:Standard 830 Breadboard, F.Cu at (-17.8, 19.8)
