File: Caon-Handwired-Prototype.kicad_pcb (KiCad board)
At the start: 6 copper layers, 40 parts, among them J1 OLED_128x32, SW4 EC11 ENCODER 1, SW8 EC11 ENCODER 1, U1 74HC595, U2 74HC595, U3 SuperMini nRF52840

Commit message: Update
Parts:
- removed REF** (x6): MX_Solder_1.00u, ScottoKeebs_Scotto:MX_Solder_1.00u
- removed REF**: OLED_128x32, ScottoKeebs_Components:OLED_128x32
- removed the SW4 at (236.9, 90.8)
- removed the SW4 at (236.9, 71.7)
- removed the U3 at (236.9, 41.5)
