File: Caon-Handwired-Schematic.kicad_pcb (KiCad board)
At the start: 6 copper layers, 30 parts, among them J1 OLED_128x32, SW4 EC11 ENCODER 1, SW8 EC11 ENCODER 1, U1 74HC595, U2 74HC595, U3 SuperMini nRF52840

Commit message: Update
Parts:
- removed D1, D2, D3, D4, D5, D6, D7, D8, S_D1, S_D2, S_D3, S_D4: ~, Caon_Footprint:D_DO-35_SOD27_P2.54mm_Caon65
- removed ENC_R1, ENC_R2, ENC_R3, ENC_R4, OLD_R1, OLD_R2: 10k, Resistor_THT:R_Axial_DIN0204_L3.6mm_D1.6mm_P2.54mm_Vertical
- removed J1: OLED_128x32, ScottoKeebs_Components:OLED_128x32
- removed SW1, SW2, SW3, SW5, SW6, SW7: ~, Caon_Footprint:SW_PUSH_6mm
- removed SW4, SW8: EC11 ENCODER 1, PCM_marbastlib-various:ROT_Alps_EC11E-Switch
- removed U1, U2: 74HC595, Package_DIP:DIP-16_W7.62mm
- removed U3: SuperMini nRF52840, Caon_Footprint:SuperMini_NiceNano_USBdn
Routing:
- net GND: track 414.8 -> 0.00 mm, vias 4 -> 0
- net +3V3: track 365.8 -> 0.00 mm, vias 8 -> 0
- net R1: track 198.1 -> 0.00 mm, vias 3 -> 0
- net R0: track 191.5 -> 0.00 mm, vias 3 -> 0
- net ENC2_A: track 175.7 -> 0.00 mm, vias 1 -> 0
- net ENC2_B: track 152.8 -> 0.00 mm, vias 1 -> 0
- net ENC1_A: track 112.3 -> 0.00 mm, vias 2 -> 0
- net ENC1_B: track 102.7 -> 0.00 mm, vias 2 -> 0
- net SCK: track 91.4 -> 0.00 mm
- net CS: track 83.2 -> 0.00 mm
- net Net-(S_D1-A): track 79.2 -> 0.00 mm
- net Net-(S_D2-A): track 69.9 -> 0.00 mm
- net Net-(S_D3-A): track 65.0 -> 0.00 mm
- net Net-(S_D4-A): track 58.4 -> 0.00 mm
- net MOSI: track 48.3 -> 0.00 mm
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